File: mainboard-v02/Avionics.sch (KiCad schematic (older format))
At the start: 35 parts, among them J8 Conn_01x03, SW1 KMR231NG LFS, U1 MAX708RESA-T, U2 ATSAMD51J20A-AU, U3 LSM9DS1, Y1 32.768kHz

Commit message: fixing bold font and adding schematic pdf of v02
Parts:
- C1, C10, C11, C13, C14, C15, C2, C4: symbol mainboard:CAP_CERAMIC0603_NO-Adafruit_Feather_M4_Express-eagle-import-lab64_SAM32-rescue-SAMD-10-rescue-SAM32-rescue -> mainboard:CAP_CERAMIC0603_NO
- C12, C16: symbol mainboard:CAP_CERAMIC0805-NOOUTLINE-Adafruit_Feather_M4_Express-eagle-import-lab64_SAM32-rescue-SAMD-10-rescue-SAM32-re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 -> mainboard:CAP_CERAMIC0805-NOOUTLINE
- D1: symbol mainboard:LED0805_NOOUTLINE-Adafruit_Feather_M4_Express-eagle-import-lab64_SAM32-rescue-SAMD-10-rescue-SAM32-rescue -> mainboard:LED0805_NOOUTLINE
- L1: symbol mainboard:INDUCTOR-Adafruit_Feather_M4_Express-eagle-import-lab64_SAM32-rescue-SAMD-10-rescue-SAM32-rescue -> mainboard:INDUCTOR
- SW1: symbol mainboard:SWITCH_TACT_SMT4.6X2.8-Adafruit_Feather_M4_Express-eagle-import-lab64_SAM32-rescue-SAMD-10-rescue-SAM32-rescue -> mainboard:SWITCH_TACT_SMT4.6X2.8
- U2: symbol mainboard:ATSAMD51J20A-AU-ATSAMD51J20A-AU-lab64_SAM32-rescue-lab64_SAM32-rescue-SAMD-10-rescue-SAM32-rescue -> mainboard:ATSAMD51J20A-AU-ATSAMD51J20A-AU
Other:
- moved on the sheet: C3, C5, C6, C7, C8, C9, J8, R1, R2, R3, R4, R42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

Commit message: mainboard-v02 with RFM98PW
Parts:
- removed J8: Conn_01x03, Connector_PinHeader_2.54mm:PinHeader_1x03_P2.54mm_Vertical, symbol Connector_Generic:Conn_01x03
- added H1, H2, H3, H4: MountingHole_Pad, MountingHole:MountingHole_3.2mm_M3_DIN965_Pad, symbol Mechanical:MountingHole_Pad
- added J10: Conn_01x03, Connector_PinHeader_2.54mm:PinHeader_1x03_P2.54mm_Vertical, symbol Connector_Generic:Conn_01x03
- added J8: Conn_01x09, Connector_PinHeader_2.54mm:PinHeader_1x09_P2.54mm_Vertical, symbol Connector_Generic:Conn_01x09
- added J9: Conn_01x05, Connector_PinHeader_2.54mm:PinHeader_1x05_P2.54mm_Vertical, symbol Connector_Generic:Conn_01x05
- C1, C10, C11, C13, C14, C15, C2, C4: symbol mainboard:CAP_CERAMIC0603_NO -> mainboard:CAP_CERAMIC0603_NO-Adafruit_Feather_M4_Express-eagle-import-lab64_SAM32-rescue-SAMD-10-rescue-SAM32-rescue
- C12, C16: symbol mainboard:CAP_CERAMIC0805-NOOUTLINE -> mainboard:CAP_CERAMIC0805-NOOUTLINE-Adafruit_Feather_M4_Express-eagle-import-lab64_SAM32-rescue-SAMD-10-rescue-SAM32-re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
- D1: symbol mainboard:LED0805_NOOUTLINE -> mainboard:LED0805_NOOUTLINE-Adafruit_Feather_M4_Express-eagle-import-lab64_SAM32-rescue-SAMD-10-rescue-SAM32-rescue
- L1: symbol mainboard:INDUCTOR -> mainboard:INDUCTOR-Adafruit_Feather_M4_Express-eagle-import-lab64_SAM32-rescue-SAMD-10-rescue-SAM32-rescue
- SW1: symbol mainboard:SWITCH_TACT_SMT4.6X2.8 -> mainboard:SWITCH_TACT_SMT4.6X2.8-Adafruit_Feather_M4_Express-eagle-import-lab64_SAM32-rescue-SAMD-10-rescue-SAM32-rescue
- U1: value MAX708RESA-T -> MAX706RS-T
- U2: symbol mainboard:ATSAMD51J20A-AU-ATSAMD51J20A-AU -> mainboard:ATSAMD51J20A-AU-ATSAMD51J20A-AU-lab64_SAM32-rescue-lab64_SAM32-rescue-SAMD-10-rescue-SAM32-rescue
Connections:
- net labels added: CS_RF, PA16, PA18, PA19, PA20, PA22, PB14, PB15, PB16, PB17, PB22, PB23, RF_IO0, RF_IO1, RF_RST
- net labels removed: CS1, CS2, CS3, CS4, DRDY1, DRDY2, DRDY3, DRDY4, RF_IO2, RF_NIRQ, RF_SDN, SPI_CS_RFM
- wire segments 170 -> 191
Other:
- note added: "Avionics"
- note added: "Breakout Pins"
- note added: "Mounting Holes"
- note removed: "CAN Rx"
- note removed: "TC4"
- note removed: "TC7"
- moved on the sheet: C3, C5, C6, C7, C8, C9, R1, R2, R3, R4, R42, R43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
