File: mainboard-v02/RF_and_GPS.sch (KiCad schematic (older format))
At the start: 12 parts, among them J5 Conn_Coaxial, J6 Conn_Coaxial, J7 Conn_Coaxial, U10 XTB-40, U11 XTB-40, U12 XTB-40, U13 EP2W+, U14 S1216V8, U15 RFM23BP, U9 XTB-40

Commit message: fixing bold font and adding schematic pdf of v02
Other:
- note added: "Science Payloads"
- note removed: "Modifications are currently needed\nto the module for radiation tolerance"
- note removed: "Sensor Modules"
- moved on the sheet: J5, J6, J7, U10, U11, U12, U13, U9

Commit message: mainboard-v02 with RFM98PW
Parts:
- removed JP7: JUMPER-PAD-3-2OF3_NC_BY_TRACE_SMALL, kmb-test:PAD-JUMPER-3-2OF3_NC_BY_TRACE_YES_SILK_FULL_BOX, symbol mainboard:JUMPER-PAD-3-2OF3_NC_BY_TRACE_SMALL
- removed U15: RFM23BP, kmb-test:RFM23BP, symbol mainboard:RFM23BP
- added J11: Conn_01x02, Connector_PinHeader_2.54mm:PinHeader_1x02_P2.54mm_Vertical, symbol Connector_Generic:Conn_01x02
- added R46, R47, R48: 0, Resistor_SMD:R_0603_1608Metric, symbol mainboard:10KOHM-1_10W-1%(0603)0603
- added U23: RFM98PW, custom-footprints:RFM98PW, symbol symbols:RFM98PW
Connections:
- net labels added: CS_RF, PA18, PA19, PA20, PA22, PB16, PB17, PB22, PB23, RF_IO0, RF_IO1, RF_IO5, RF_RST
- net labels removed: CS1, CS2, CS3, CS4, DRDY1, DRDY2, DRDY3, DRDY4, RF_NIRQ, RF_SDN, SPI_CS_RFM
- wire segments 68 -> 67
Other:
- note added: "DNI"
- note added: "HopeRF RFM98PW module at 3.3V"
- note added: "Payload Modules"
- note added: "Radio, GPS, Payloads"
- note added: "Radio\nVCC"
- note removed: "HopeRF RFM23B module at 3.3V"
- note removed: "Science Payloads"
- moved on the sheet: J5, J6, J7, R24, U10, U11, U12, U13, U9
