File: mainboard-v02/mainboard.sch (KiCad schematic (older format))
At the start: 0 parts

Commit message: fixing bold font and adding schematic pdf of v02
Other:
- note removed: "DRDY pins on XTB\nADD BREAKOUT AREA\nCONFIRM GPS SCHEME\n\n"
- note removed: "TO DO"
Changed lines of the file:
@@
 EESchema Schematic File Version 4
-LIBS:mainboard
 EELAYER 29 0
 EELAYER END
@@
 F1 "Burn_Wires.sch" 50
 $EndSheet
-Text Notes 1850 1850 0    100  ~ 0
-TO DO
-Text Notes 1850 2550 0    100  ~ 0
-DRDY pins on XTB\nADD BREAKOUT AREA\nCONFIRM GPS SCHEME\n\n
 $EndSCHEMATC
