File: mainboard-v02/mainboard.kicad_pcb (KiCad board)
At the start: 4 copper layers, 90.2 x 95.9 mm, 152 parts, among them J1 503182-1852, J10 Conn_01x03, J11 Conn_01x02, J2 Conn_01x05, J3 10118194-0001LF, J4 DCJ0303, J5 Conn_Coaxial, J6 Conn_Coaxial, J7 Conn_Coaxial, J8 Conn_01x09, J9 Conn_01x05, Q1 IRLML2803, Q2 2N5088, Q3 2N5088, Q4 IRLML2803, Q5 IRLML2803, Q6 IRLML2803, Q7 IRLML2803, Q8 IRLML2803, SW1 KMR231NG LFS, U1 MAX706RS-T, U10 XTB-40, U11 XTB-40, U12 XTB-40, U13 EP2W+, U14 S1216V8, U16 PE014006, U17 PE014006, U18 NDS8434, U19 NDS8434, U2 ATSAMD51J20A-AU, U20 NDS8434, U21 NDS8434, U22 NDS8434, U23 RFM98PW, U3 LSM9DS1, U4 MAX4372TEUK+T, U5 TPS54226PWPRPWP14_2P31X2P46-L, U6 LTC4121, U7 NDS8434, U8 MR25H40MDF, U9 XTB-40, Y1 32.768kHz

Commit message: fixing flux capacitor layout
Parts:
- removed the G*** at (157.5, 120.4) (x2)
- removed U1: MAX706RS-T, Package_SO:SO-8_3.9x4.9mm_P1.27mm
- added G*** (x2): LOGO, LOGO, F.Cu at (157.5, 120.4)
