File: mainboard-v03/Power_USB-BAK.sch (KiCad schematic (older format))
At the start: 53 parts, among them Q1 IRLML2803, U17 BQ25883RGER, U4 ADM1176-1ARMZ-R7, U5 TPS54226PWPRPWP14_2P31X2P46-L, U6 LTC4121, U7 NDS8434

Commit message: mainboardv3 clean up
Parts:
- added C33, C34, C38, C39: 1uF, Capacitor_SMD:C_0603_1608Metric, symbol Device:C_Small
- added C35: 3.9nF, Capacitor_SMD:C_0603_1608Metric, symbol Device:C_Small
- added C36, C37: 0.1uF, Capacitor_SMD:C_0603_1608Metric, symbol Device:C_Small
- added C40: 10uF, Capacitor_SMD:C_0603_1608Metric, symbol Device:C_Small
- added D5: GREEN LED, LED_SMD:LED_0603_1608Metric, symbol mainboard:LED0805_NOOUTLINE-Adafruit_Feather_M4_Express-eagle-import-lab64_SAM3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
- added L4: 2.2uH, custom-footprints:XFL4030472MEB, symbol Device:L
- added Q3: AS3423B, Package_TO_SOT_SMD:SOT-23, symbol Transistor_FET:BS250
- added R31: 10K, Resistor_SMD:R_0603_1608Metric, symbol Device:R_US
- added R34: 3.3K, Resistor_SMD:R_0603_1608Metric, symbol Device:R_US
- added R35: 1K, Resistor_SMD:R_0603_1608Metric, symbol Device:R_US
- added U17: MAX14748AEWW+, custom-footprints:MAX14748AEWW&plus_mod, symbol symbols:MAX14748AEWW+
- C19, C20: value 100uF -> 220UF
- C32: value 3.3nF -> 3.9nF
- L?: renamed from L4; PN DFE252012F-1R0M=P2 -> XFL4020-222ME
- R?: renamed from R34; value 5.23K -> 2.2K
- renumbered C36 to C?, C37 to C?, C39 to C?, C34 to C?, C33 to C?, C35 to C?, C38 to C?, D5 to D?, R31 to R?, R35 to R?, R36 to R?, U17 to U?
Connections:
- net labels added: 3V3_IN, CHGIN, LX, USB_CC1, USB_CC2, VCCINT
- wire segments 191 -> 255
- no-connect marks 4 -> 14
Other:
- note added: "USB-C Power Delivery w/ Battery Charger (2-cell)"
- note removed: "USB (Boost) Charging for 2-cell Li-Ion"
- moved on the sheet: C?, D?, L?, R?, U?
