File: mainboard-v03/mainboard.kicad_pcb (KiCad board)
At the start: 4 copper layers, 90.2 x 95.9 mm, 152 parts, among them J1 503182-1852, J10 Conn_01x03, J11 Conn_01x02, J2 Conn_01x05, J3 10118194-0001LF, J4 DCJ0303, J5 Conn_Coaxial, J6 Conn_Coaxial, J7 Conn_Coaxial, J8 Conn_01x09, J9 Conn_01x05, Q1 IRLML2803, Q2 2N5088, Q3 2N5088, Q4 IRLML2803, Q5 IRLML2803, Q6 IRLML2803, Q7 IRLML2803, Q8 IRLML2803, SW1 KMR231NG LFS, U1 MAX706RS-T, U10 XTB-40, U11 XTB-40, U12 XTB-40, U13 EP2W+, U14 S1216V8, U16 PE014006, U17 PE014006, U18 NDS8434, U19 NDS8434, U2 ATSAMD51J20A-AU, U20 NDS8434, U21 NDS8434, U22 NDS8434, U23 RFM98PW, U3 LSM9DS1, U4 MAX4372TEUK+T, U5 TPS54226PWPRPWP14_2P31X2P46-L, U6 LTC4121, U7 NDS8434, U8 MR25H40MDF, U9 XTB-40, Y1 32.768kHz

Commit message: mainboardv3 clean up
Parts:
- removed the G*** at (153.2, 120.4)
- removed the G*** at (157.5, 120.4) (x2)
- removed Q3: 2N5088, mainboard:SOT23
- removed Q6, Q7, Q8: IRLML2803, mainboard:SOT-23
- removed R41: 100k, Resistor_SMD:R_0603_1608Metric
- removed R43: 0, Resistor_SMD:R_0603_1608Metric
- removed U21, U22: NDS8434, custom-footprints:NDS8434
- added ?: , , F.Cu at (158.5, 56.6)
- added C24: 0.1uF, Capacitor_SMD:C_0603_1608Metric, F.Cu at (170.5, 69.3)
- added C31: 22uF, Capacitor_SMD:C_0603_1608Metric, F.Cu at (170.5, 71.5)
- added C32: 3.9nF, Capacitor_SMD:C_0603_1608Metric, F.Cu at (160.1, 91.2)
- added C33: 1uF, Capacitor_SMD:C_0603_1608Metric, B.Cu at (148.0, 64.4)
- added C34: 4.7uF, Capacitor_SMD:C_0603_1608Metric, F.Cu at (153.2, 67.2)
- added C35: 10uF, Capacitor_SMD:C_0603_1608Metric, B.Cu at (148.7, 67.0)
- added C36: 47nF, Capacitor_SMD:C_0603_1608Metric, F.Cu at (153.2, 68.5)
- added C37: 22uF, Capacitor_SMD:C_0603_1608Metric, B.Cu at (153.4, 70.6)
- added C38: 22uF, Capacitor_SMD:C_0603_1608Metric, B.Cu at (151.7, 70.6)
- added C39: 10uF, Capacitor_SMD:C_0603_1608Metric, B.Cu at (155.3, 70.6)
- added G***: LOGO, LOGO, F.Cu at (157.5, 120.4)
- added G***: LOGO, LOGO, F.Cu at (153.9, 120.9)
- added G***: LOGO, LOGO, F.Cu at (158.5, 120.7)
- added G***: LOGO, LOGO, F.Cu at (163.2, 130.5)
- added J12: Conn_Coaxial, Connector_Coaxial:SMA_Amphenol_901-144_Vertical, F.Cu at (183.0, 135.7)
- added J13: USB_C_Receptacle_USB2.0, custom-footprints:USB_C_Receptacle_XKB_U262-161N-4BVC11, F.Cu at (148.1, 55.0)
- added L4: 1uH, custom-footprints:XFL4030472MEB, B.Cu at (148.7, 71.1)
- added REF**: Gauge_10mm_Type1_SilkScreenTop, Calibration_Scale:Gauge_10mm_Type1_SilkScreenTop, F.Cu at (99.8, 83.3)
- added REF**: Fiducial_1mm_Mask2mm, Fiducial:Fiducial_1mm_Mask2mm, B.Cu at (186.4, 54.4)
- added REF**: Fiducial_1mm_Mask2mm, Fiducial:Fiducial_1mm_Mask2mm, F.Cu at (186.4, 54.4)
- added REF**: Fiducial_1mm_Mask2mm, Fiducial:Fiducial_1mm_Mask2mm, B.Cu at (100.8, 54.9)
- added REF**: Fiducial_1mm_Mask2mm, Fiducial:Fiducial_1mm_Mask2mm, F.Cu at (100.8, 54.9)
- added REF**: Fiducial_1mm_Mask2mm, Fiducial:Fiducial_1mm_Mask2mm, B.Cu at (100.3, 146.6)
- added REF**: Fiducial_1mm_Mask2mm, Fiducial:Fiducial_1mm_Mask2mm, F.Cu at (100.3, 146.6)
- added Ref**: Val**, custom-footprints:sun, F.Cu at (115.2, 147.5)
- added Ref**: Val**, custom-footprints:sun, B.Cu at (187.3, 123.6)
- added Ref**: Val**, custom-footprints:sun, B.Cu at (174.5, 146.8)
- added Ref**: Val**, custom-footprints:sun, B.Cu at (137.9, 146.8)
- added Ref**: Val**, custom-footprints:sun, B.Cu at (115.2, 146.9)
- added Ref**: Val**, custom-footprints:sun, B.Cu at (121.0, 54.0)
- added Ref**: Val**, custom-footprints:sun, B.Cu at (187.2, 100.3)
- added Ref**: Val**, custom-footprints:sun, B.Cu at (99.7, 89.8)
- added Ref**: Val**, custom-footprints:layers, F.Cu at (108.2, 148.6)
- added Ref**: Val**, custom-footprints:mainboard_version, B.Cu at (133.3, 54.1)
- added Ref**: Val**, custom-footprints:mainboard_version, F.Cu at (132.3, 54.1)
- added Ref**: Val**, custom-footprints:sun, F.Cu at (137.9, 147.5)
- added Ref**: Val**, custom-footprints:flame, F.Cu at (187.6, 97.8)
- added Ref**: Val**, custom-footprints:flame, F.Cu at (99.3, 92.4)
- added Ref**: Val**, custom-footprints:flame, B.Cu at (187.3, 97.8)
- added Ref**: Val**, custom-footprints:flame, B.Cu at (99.6, 92.3)
- added Ref**: Val**, custom-footprints:pycubed_logo, B.Cu at (142.7, 120.5)
- added Ref**: Val**, custom-footprints:pycubed_logo, F.Cu at (156.7, 123.2)
- added Ref**: Val**, custom-footprints:XYZ, F.Cu at (179.1, 112.8)
- added Ref**: Val**, custom-footprints:sun, F.Cu at (174.5, 147.3)
- added Ref**: Val**, custom-footprints:sun, F.Cu at (187.6, 123.3)
- added Ref**: Val**, custom-footprints:sun, F.Cu at (165.2, 53.9)
- added Ref**: Val**, custom-footprints:sun, F.Cu at (121.0, 53.3)
- added Ref**: Val**, custom-footprints:sun, F.Cu at (187.6, 100.4)
- added Ref**: Val**, custom-footprints:sun, F.Cu at (99.3, 89.9)
- added Ref**: Val**, custom-footprints:sun, B.Cu at (165.2, 53.4)
- added U15: RFM9xBreakout, RF_Module:HOPERF_RFM9XW_SMD, B.Cu at (168.6, 129.4)
- added U24: RFM98PW, custom-footprints:RFM98PW, B.Cu at (168.1, 119.9)
- C29: value 2.2uF -> 4.7uF
- D3: value MBR120 -> ESDA25P35; footprint custom-footprints:D_SOD-123 -> custom-footprints:ESDA8P801U1M
- D5: value SBR2A40P1Q-7 -> GREEN LED; footprint mainboard:PWRDI-123 -> LED_SMD:LED_0603_1608Metric
- H1: footprint MountingHole:MountingHole_3.2mm_M3_ISO7380_Pad -> MountingHole:MountingHole_3.2mm_M3_DIN965_Pad
- J10: value Conn_01x03 -> Conn_01x05; footprint Connector_PinHeader_2.54mm:PinHeader_1x03_P2.54mm_Vertical -> Connector_PinHeader_2.54mm:PinHeader_1x05_P2.54mm_Vertical
- J3: value 10118194-0001LF -> Conn_01x01; footprint mainboard:FRAMATOME_10118194-0001LF -> Connector_PinHeader_2.54mm:PinHeader_1x01_P2.54mm_Vertical
- J4: value DCJ0303 -> 10118194-0001LF; footprint mainboard:DCJ0303 -> custom-footprints:10118194-0001LF; moved to B.Cu
- J5, J6: moved to B.Cu
- R10: value 40.9K -> 40.2K
- R26, R31: value 10k -> 1K
- R29: value 10k -> 0
- R30: value 10k -> 10K
- R34: value 4.7k -> 5.23K; moved to B.Cu
- R35: value 4.7k -> 30.1K; moved to B.Cu
- R36: value 4.7k -> 383; moved to B.Cu
- R39, R40: value 100k -> 5.1k; moved to B.Cu
- R42: value 0 -> 10k; moved to F.Cu
- R5: value 2.2K -> 1K
- U17: value PE014006 -> BQ25883RGER; footprint mainboard:RELAY5-PE_CO -> custom-footprints:QFN50P400X400X100-25N-D; moved to B.Cu
- U2: footprint ATSAMD51J20A-AU:QFP50P1200X1200X120-64N -> custom-footprints:QFP50P1200X1200X120-64N
- U20: value NDS8434 -> RFM9xBreakout; footprint custom-footprints:NDS8434 -> RF_Module:HOPERF_RFM9XW_SMD
- U3: footprint mainboard:LGA24-8X4 -> custom-footprints:LSM9DS1
- U4: value MAX4372TEUK+T -> ADM1176-1ARMZ-R7; footprint mainboard:21-0057F -> custom-footprints:ADM1176-1ARMZ-R7
- moved J4 83.5 mm to (147.5, 54.5)
- moved R34 82.5 mm to (157.0, 62.9), turned to 0 degrees
- moved R39 80.3 mm to (148.1, 63.1), turned to 180 degrees
- moved R40 76.9 mm to (148.1, 61.8), turned to 0 degrees
- moved R31 76.9 mm to (157.6, 56.4), turned to 270 degrees
- moved R35 73.2 mm to (161.2, 62.9), turned to 180 degrees
- moved U17 72.7 mm to (152.4, 66.3), turned to 270 degrees
- moved R36 70.4 mm to (157.5, 65.3), turned to 180 degrees
- moved D5 58.1 mm to (159.6, 56.4), turned to 270 degrees
- moved R29 54.6 mm to (164.8, 97.3), turned to 90 degrees
- moved J3 41.0 mm to (171.3, 88.3), turned to 0 degrees
- moved R30 39.0 mm to (166.4, 94.5), turned to 90 degrees
- moved JP15 32.1 mm to (184.4, 126.0), turned to 90 degrees
- moved C29 24.1 mm to (154.1, 56.4), turned to 90 degrees
- moved R26 20.6 mm to (166.4, 91.2), turned to 90 degrees
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Connections:
- net RF_IO5 renamed Net-(U23-Pad15)
- C22 pad 1: Net-(C22-Pad1) -> /Power/VCHRG_IN
- C25 pad 2: Net-(C25-Pad2) -> /Power/VCHRG_IN
- C29 pad 1: /Connectors/VBATT_IN -> VBUS_IN
- C29 pad 2: GND -> GNDREF
- C4 pad 2: ~RESET -> /Avionics/~RESET
- D2 pad C: Net-(C22-Pad1) -> /Power/VCHRG_IN
- D3 pad 1: /Connectors/VBATT_IN -> GNDREF
- D3 pad 2: Net-(D3-Pad2) -> VBUS_IN
- J10 pad 2: PB15 -> AIN4
- J10 pad 3: PB14 -> AIN5
- J3 pad 1: Net-(D3-Pad2) -> THM
- J4 pad 1: VBATT -> VBUS_IN
- J4 pad 2: Net-(J4-Pad2) -> USB_D-
- J4 pad 3: Net-(J4-Pad2) -> USB_D+
- J7 pad 1: Net-(J7-Pad1) -> RF1_ANT
- J9 pad 5: PA16 -> PA17
- JP13 pad 3: /Burn Wires/VBURN3 -> Net-(JP13-Pad3)
- JP14 pad 3: /Burn Wires/VBURN4 -> Net-(JP14-Pad3)
- JP15 pad 3: /Burn Wires/VBURN5 -> Net-(JP15-Pad3)
- JP2 pad 1: /Connectors/VBATT_IN -> VCHRG
- JP2 pad 2: Net-(J4-Pad2) -> GNDREF
- JP3 pad 1: /Connectors/VBATT_IN -> VCHRG
- JP3 pad 2: Net-(J4-Pad2) -> GNDREF
- JP4 pad 1: Net-(J4-Pad2) -> GNDREF
- JP5 pad 2: /Connectors/VBATT_IN -> VCHRG
- L3 pad 2: Net-(C25-Pad2) -> /Power/VCHRG_IN
- R10 pad 2: Net-(C22-Pad1) -> /Power/VCHRG_IN
- R11 pad 2: Net-(C22-Pad1) -> /Power/VCHRG_IN
- R26 pad 1: BURN_RELAY_B -> Net-(R26-Pad1)
- R26 pad 2: GND -> VBATT
- R29 pad 1: ENAB_BURN3 -> Net-(R29-Pad1)
- R29 pad 2: GND -> Net-(R29-Pad2)
- R3 pad 2: ~RESET -> /Avionics/~RESET
- R30 pad 1: ENAB_BURN4 -> Net-(R29-Pad1)
- R30 pad 2: GND -> VBATT
- R31 pad 1: ENAB_BURN5 -> Net-(D5-Pad1)
- R31 pad 2: GND -> VBUS_IN
- R34 pad 1: Net-(Q6-Pad1) -> VBUS_IN
- R34 pad 2: ENAB_BURN3 -> THM
- R35 pad 1: Net-(Q7-Pad1) -> GNDREF
- R35 pad 2: ENAB_BURN4 -> THM
- R36 pad 1: Net-(Q8-Pad1) -> GNDREF
- R36 pad 2: ENAB_BURN5 -> Net-(R36-Pad2)
- R39 pad 1: Net-(Q6-Pad3) -> GNDREF
- R39 pad 2: /Burn Wires/VBURN_B_IN -> USB_CC2
- R40 pad 1: Net-(Q7-Pad3) -> GNDREF
- R40 pad 2: /Burn Wires/VBURN_B_IN -> USB_CC1
- R42 pad 1: 3.3V -> /Avionics/~RESET
- R44 pad 2: /Avionics/SDA -> SDA
- R45 pad 2: /Avionics/SCL -> SCL
- SW1 pad A: ~RESET -> /Avionics/~RESET
- SW1 pad A': ~RESET -> /Avionics/~RESET
- U1 pad 1: Net-(R42-Pad2) -> Net-(U1-Pad1)
- U1 pad 2: Net-(R42-Pad2) -> 3.3V
- U1 pad 7: ~RESET -> Net-(R42-Pad2)
- U1 pad 8: ~RESET -> Net-(R42-Pad2)
- U17 pad 1: VBATT -> USB_D-
- U17 pad 11: /Burn Wires/VBURN_B_IN -> Net-(C34-Pad1)
- U17 pad 12: GND -> Net-(C36-Pad2)
- U17 pad 14: VBATT -> VCHRG
- U17 pad 5: Net-(D5-PadA) -> SCL
- U2 pad 10: ENAB_BURN3 -> RF2_BUSY
- U2 pad 12: ENAB_BURN4 -> RF2_CS
- U2 pad 13: I_BATT -> AIN4
- U2 pad 14: BURN_RELAY_B -> AIN5
- U2 pad 25: /Avionics/SDA -> SDA
- U2 pad 26: /Avionics/SCL -> SCL
- U2 pad 27: PB14 -> RF2_RST
- U2 pad 28: PB15 -> BURN_RELAY_A
- U2 pad 35: PA16 -> Net-(U2-Pad35)
- U2 pad 36: BURN_RELAY_A -> PA17
- U2 pad 5: ENAB_BURN5 -> RF1_IO4
- U2 pad 52: ~RESET -> /Avionics/~RESET
- U2 pad 59: CS_RF -> RF1_CS
- U2 pad 6: RF_IO0 -> RF1_IO0
- U2 pad 61: RF_RST -> RF1_RST
- U2 pad 9: RF_IO1 -> RF2_IO1
- U20 pad 1: /Burn Wires/VBURN_B_IN -> GND
- U20 pad 2: /Burn Wires/VBURN_B_IN -> MISO
- U20 pad 3: /Burn Wires/VBURN_B_IN -> MOSI
- U20 pad 4: Net-(Q6-Pad3) -> SCK
- U20 pad 5: /Burn Wires/VBURN3 -> RF1_CS
- U20 pad 6: /Burn Wires/VBURN3 -> RF1_RST
- U20 pad 7: /Burn Wires/VBURN3 -> Net-(U20-Pad7)
- U20 pad 8: /Burn Wires/VBURN3 -> GND
- U23 pad 1: Net-(J7-Pad1) -> RF1_ANT
- U23 pad 13: CS_RF -> RF1_CS
- U23 pad 14: RF_RST -> RF1_RST
- U23 pad 4: Net-(U23-Pad4) -> RF1_IO4
- U23 pad 6: RF_IO0 -> RF1_IO0
- U23 pad 7: RF_IO1 -> RF1_IO1
- U23 pad 8: RF_IO2 -> RF1_IO2
- U3 pad 2: /Avionics/SCL -> SCL
- U3 pad 4: /Avionics/SDA -> SDA
- U4 pad 1: GND -> VBATT
- U4 pad 2: I_BATT -> /Power/VREG_IN
- U4 pad 3: 3.3V -> Net-(R26-Pad1)
- U4 pad 4: VBATT -> GND
- U4 pad 5: /Power/VREG_IN -> Net-(C32-Pad2)
- U5 pad 7: VBATT -> Net-(R29-Pad1)
- U6 pad P$3: Net-(C22-Pad1) -> /Power/VCHRG_IN
- U6 pad P$4: Net-(C25-Pad2) -> /Power/VCHRG_IN
Routing:
- net Net-(J4-Pad2): track 95.9 -> 0.00 mm
- net VBATT: track 165.6 -> 73.0 mm
- net /Burn Wires/VBURN_B_IN: track 69.7 -> 0.00 mm, vias 3 -> 0
- net RF1_IO0: track 0.00 -> 68.1 mm, vias 0 -> 3
- net SCL: track 0.00 -> 65.8 mm, vias 0 -> 4
- net SCK: track 109.8 -> 175.4 mm, vias 3 -> 4
- net SDA: track 0.00 -> 65.5 mm, vias 0 -> 4
- net MOSI: track 108.7 -> 170.0 mm, vias 4 -> 5
- net MISO: track 112.5 -> 173.8 mm, vias 3 -> 4
- net RF2_RST: track 0.00 -> 51.3 mm, vias 0 -> 2
- net THM: track 0.00 -> 42.5 mm, vias 0 -> 1
- net RF2_CS: track 0.00 -> 42.2 mm, vias 0 -> 2
- net RF1_RST: track 0.00 -> 42.2 mm, vias 0 -> 2
- net RF1_IO4: track 0.00 -> 41.7 mm, vias 0 -> 2
- net ENAB_BURN4: track 41.2 -> 0.00 mm, vias 2 -> 0
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- added copper zone on B.Cu, net (none)
- added copper zone on F.Cu, net (none)
- added copper zone on F.Cu, net /Power/VCHRG_IN
- added copper zone on B.Cu, net GNDREF
- added copper zone on F.Cu, net VCHRG
- removed copper zone on F.Cu, net /Burn Wires/VBURN3
- removed copper zone on F.Cu, net /Burn Wires/VBURN4
- removed copper zone on F.Cu, net /Burn Wires/VBURN5
- removed copper zone on F.Cu, net /Burn Wires/VBURN_B_IN
- removed copper zone on F.Cu, net /Connectors/VBATT_IN
- removed copper zone on F.Cu, net Net-(C22-Pad1)
- removed copper zone on F.Cu, net Net-(C25-Pad2)
- removed copper zone on Route15, net Net-(J4-Pad2)
Other:
- net class Default: clearance 0.1524 -> 0.127; via_dia 0.6 -> 0.5842; via_drill 0.4 -> 0.381
- rule trace_clearance: 0.1524 -> 0.127
- rule trace_min: 0.2 -> 0.127
- rule via_min_drill: 0.3 -> 0.381
- rule via_min_size: 0.4 -> 0.5842
- board text added: "AIN4"
- board text added: "AIN5"
- board text added: "ANT"
- board text added: "BATT THERM"
- board text added: "BURN1"
- board text added: "BURN2"
- board text added: "CHRG LED"
- board text added: "CS"
- board text added: "IO0"
- board text added: "IO1"
- board text added: "IO2"
- board text added: "IO3"
- board text added: "IO4"
- board text added: "IO5"
- board text added: "MODULAR RADIO #1"
- board text added: "MODULAR RADIO #2"
- board text added: "PA17"
- board text added: "RADIO #1"
- board text added: "RADIO #2"
- board text added: "RADIO VDD"
- board text added: "RST"
- board text added: "VDD"
- board text added: "WDT EN"
- board text added: "v3"
- board text removed: "4.5V TO 18V"
- board text removed: "ANTENNA 1"
- board text removed: "ANTENNA 2"
- board text removed: "DEPOLY 1"
- board text removed: "DEPOLY 2"
- board text removed: "DEPOLY 3"
- board text removed: "GPS"
- board text removed: "GPS ~RST"
- board text removed: "GPS1"
- board text removed: "GPS2"
- board text removed: "JTAG"
- board text removed: "ON/OFF"
- board text removed: "PA16"
- board text removed: "PB14"
- board text removed: "PB15"
- board text removed: "RADIO"
- board text removed: "RADIO VCC"
- board text removed: "RFM98PW"
- board text removed: "SOLAR"
- board text removed: "VBATT"
- board text removed: "VBURN"
- board text removed: "VSOL"
- board text removed: "WDT"
