File: mainboard-v04/Burn_Wires.sch (KiCad schematic (older format))
At the start: 22 parts, among them Q2 2N5088, Q4 IRLML2803, Q5 IRLML2803, U16 PE014006, U18 NDS8434, U19 NDS8434

Commit message: adding mainbaordv04 layout and BOM
Parts:
- D4: Flight (none) -> SBR2A40P1Q-7; Proto (none) -> SBR2A40P1Q-7
- Q4: Proto IRLML2803 -> 2302
- Q5: Flight (none) -> IRLML2803; Proto (none) -> 2302
- U19: Field4 ON Semiconductor -> (none); Field5 Unavailable -> (none); Field6 None -> (none); Field7 NDS8434 -> (none); Field8 SO-8 ON Semiconductor -> (none); Flight (none) -> NDS8434; Proto (none) -> DMP2022LSS-13
Changed lines of the file:
@@
 EESchema Schematic File Version 4
-LIBS:mainboard-cache
 EELAYER 30 0
 EELAYER END
@@
 Sheet 2 6
 Title "PyCubed Mainboard"
-Date "2019-11-27"
+Date "2020-01-08"
 Rev "v04"
-Comp "Stanford University"
+Comp ""
 Comment1 "Zac Manchester"
 Comment2 "Max Holliday"
@@
 F 2 "mainboard:SOT-23" H 6500 1600 50  0001 C CNN
 F 3 "" H 6500 1600 50  0001 C CNN
-F 4 "IRLML2803" V 6500 1600 50  0001 C CNN "Proto"
+F 4 "2302" V 6500 1600 50  0001 C CNN "Proto"
 F 5 "IRLML2803" V 6500 1600 50  0001 C CNN "Flight"
 	1    6500 1600
@@
 F 2 "mainboard:SOT-23" H 6500 2550 50  0001 C CNN
 F 3 "" H 6500 2550 50  0001 C CNN
+F 4 "IRLML2803" H 6500 2550 50  0001 C CNN "Flight"
+F 5 "2302" H 6500 2550 50  0001 C CNN "Proto"
 	1    6500 2550
 	0    1    1    0
@@
 F 2 "mainboard:PWRDI-123" H 2300 1400 50  0001 C CNN
 F 3 "" H 2300 1400 50  0001 C CNN
+F 4 "SBR2A40P1Q-7" H 2300 1400 50  0001 C CNN "Flight"
+F 5 "SBR2A40P1Q-7" H 2300 1400 50  0001 C CNN "Proto"
 	1    2300 1400
 	0    -1   -1   0
@@
 F 2 "custom-footprints:NDS8434" H 7500 2450 50  0001 L BNN
 F 3 "" H 7500 2450 50  0001 L BNN
-F 4 "ON Semiconductor" H 7500 2450 50  0001 L BNN "Field4"
-F 5 "Unavailable" H 7500 2450 50  0001 L BNN "Field5"
-F 6 "None" H 7500 2450 50  0001 L BNN "Field6"
-F 7 "NDS8434" H 7500 2450 50  0001 L BNN "Field7"
-F 8 "SO-8 ON Semiconductor" H 7500 2450 50  0001 L BNN "Field8"
+F 4 "" H 7500 2450 50  0001 L BNN "Field4"
+F 5 "" H 7500 2450 50  0001 L BNN "Field5"
+F 6 "" H 7500 2450 50  0001 L BNN "Field6"
+F 7 "" H 7500 2450 50  0001 L BNN "Field7"
+F 8 "" H 7500 2450 50  0001 L BNN "Field8"
+F 9 "NDS8434" H 7500 2450 50  0001 C CNN "Flight"
+F 10 "DMP2022LSS-13" H 7500 2450 50  0001 C CNN "Proto"
 	1    7500 2450
 	1    0    0    -1

Commit message: cleaned up v04
Parts:
- JP10: value M03POLAR_LOCK -> Conn_01x03
- JP11, JP12, JP13, JP14, JP15, JP8, JP9: value M03POLAR_LOCK -> Conn_01x03; DNI (none) -> DNI
- Q2: Proto 2N5088 -> S8050
Other:
- note added: "NOTE: Components labeled "do not install" (DNI) are not populated by default"
Changed lines of the file:
@@
 EELAYER 30 0
 EELAYER END
-$Descr User 11693 8548
+$Descr A4 11693 8268
 encoding utf-8
-Sheet 2 6
+Sheet 5 6
 Title "PyCubed Mainboard"
-Date "2020-01-08"
+Date "2020-02-10"
 Rev "v04"
-Comp ""
-Comment1 "Zac Manchester"
-Comment2 "Max Holliday"
+Comp "Max Holliday"
+Comment1 ""
+Comment2 ""
 Comment3 ""
 Comment4 ""
@@
 AR Path="/5CEC6476/A21E5090" Ref="JP11"  Part="1"
 F 0 "JP11" H 8400 1930 59  0000 L BNN
-F 1 "M03POLAR_LOCK" V 8550 750 59  0001 L BNN
+F 1 "Conn_01x03" V 8550 750 59  0001 L BNN
 F 2 "mainboard:MOLEX-1X3_LOCK" H 8500 1700 50  0001 C CNN
 F 3 "" H 8500 1700 50  0001 C CNN
+F 4 "DNI" V 8500 1700 50  0000 C CNB "DNI"
 	1    8500 1700
 	0    -1   -1   0
@@
 AR Path="/5CEC6476/056852D9" Ref="JP12"  Part="1"
 F 0 "JP12" H 8400 2880 59  0000 L BNN
-F 1 "M03POLAR_LOCK" H 8400 2350 59  0001 L BNN
+F 1 "Conn_01x03" H 8400 2350 59  0001 L BNN
 F 2 "mainboard:MOLEX-1X3_LOCK" H 8500 2650 50  0001 C CNN
 F 3 "" H 8500 2650 50  0001 C CNN
+F 4 "DNI" V 8500 2650 50  0000 C CNB "DNI"
 	1    8500 2650
 	0    -1   -1   0
@@
 AR Path="/5CEC6476/C8B46213" Ref="JP13"  Part="1"
 F 0 "JP13" H 1600 5480 59  0000 L BNN
-F 1 "M03POLAR_LOCK" H 1600 4950 59  0001 L BNN
+F 1 "Conn_01x03" H 1600 4950 59  0001 L BNN
 F 2 "mainboard:MOLEX-1X3_LOCK" H 1700 5250 50  0001 C CNN
 F 3 "" H 1700 5250 50  0001 C CNN
+F 4 "DNI" V 1700 5250 50  0000 C CNB "DNI"
 	1    1700 5250
 	0    -1   -1   0
@@
 AR Path="/5CEC6476/4861989B" Ref="JP10"  Part="1"
 F 0 "JP10" H 4850 4380 59  0000 L BNN
-F 1 "M03POLAR_LOCK" H 4850 3850 59  0000 L BNN
+F 1 "Conn_01x03" H 4850 3850 59  0000 L BNN
 F 2 "mainboard:MOLEX-1X3_LOCK" H 4950 4150 50  0001 C CNN
-F 3 "" H 4950 4150 50  0001 C CNN
+F 3 "DNI" H 4950 4150 50  0000 C CNB
 	1    4950 4150
 	1    0    0    -1
@@
 AR Path="/5CEC6476/FF5F0BF4" Ref="JP8"  Part="1"
 F 0 "JP8" H 1450 4380 59  0000 L BNN
-F 1 "M03POLAR_LOCK" H 1450 3850 59  0000 L BNN
+F 1 "Conn_01x03" H 1450 3850 59  0000 L BNN
 F 2 "mainboard:MOLEX-1X3_LOCK" H 1550 4150 50  0001 C CNN
 F 3 "" H 1550 4150 50  0001 C CNN
+F 4 "DNI" H 1550 4150 50  0000 C CNB "DNI"
 	1    1550 4150
 	1    0    0    -1
@@
 AR Path="/5CEC6476/2206741E" Ref="JP9"  Part="1"
 F 0 "JP9" H 3050 4380 59  0000 L BNN
-F 1 "M03POLAR_LOCK" H 3050 3850 59  0000 L BNN
+F 1 "Conn_01x03" H 3050 3850 59  0000 L BNN
 F 2 "mainboard:MOLEX-1X3_LOCK" H 3150 4150 50  0001 C CNN
 F 3 "" H 3150 4150 50  0001 C CNN
+F 4 "DNI" H 3150 4150 50  0000 C CNB "DNI"
 	1    3150 4150
 	1    0    0    -1
@@
 AR Path="/5CEC6476/357D3C8D" Ref="JP14"  Part="1"
 F 0 "JP14" H 3150 5530 59  0000 L BNN
-F 1 "M03POLAR_LOCK" H 3150 5000 59  0001 L BNN
+F 1 "Conn_01x03" H 3150 5000 59  0001 L BNN
 F 2 "mainboard:MOLEX-1X3_LOCK" H 3250 5300 50  0001 C CNN
 F 3 "" H 3250 5300 50  0001 C CNN
+F 4 "DNI" V 3250 5300 50  0000 C CNB "DNI"
 	1    3250 5300
 	0    -1   -1   0
@@
 AR Path="/5CEC6476/ADC4B3B7" Ref="JP15"  Part="1"
 F 0 "JP15" H 4950 5530 59  0000 L BNN
-F 1 "M03POLAR_LOCK" H 4950 5000 59  0001 L BNN
+F 1 "Conn_01x03" H 4950 5000 59  0001 L BNN
 F 2 "mainboard:MOLEX-1X3_LOCK" H 5050 5300 50  0001 C CNN
 F 3 "" H 5050 5300 50  0001 C CNN
+F 4 "DNI" V 5050 5300 50  0000 C CNB "DNI"
 	1    5050 5300
 	0    -1   -1   0
@@
 F 2 "mainboard:SOT23" H 2200 1700 50  0001 C CNN
 F 3 "" H 2200 1700 50  0001 C CNN
-F 4 "2N5088" H 2200 1700 50  0001 C CNN "Proto"
+F 4 "S8050" H 2200 1700 50  0001 C CNN "Proto"
 F 5 "2N5088" H 2200 1700 50  0001 C CNN "Flight"
 	1    2200 1700
@@
 	0    -1   -1   0
 $EndComp
-Text Notes 2700 1900 0    85   ~ 0
+Text Notes 2850 1900 0    85   ~ 0
 Power Relay A
 Text Notes 4500 800  0    85   ~ 0
@@
 	7000 2350 7000 2150
 Connection ~ 6700 2150
-Text Notes 8600 7250 0    200  ~ 0
+Text Notes 8600 6950 0    200  ~ 40
 Burn Wires
 NoConn ~ 1600 4950
@@
 NoConn ~ 3450 4050
 NoConn ~ 1850 4050
+Text Notes 7000 6500 0    65   ~ 0
+NOTE: Components labeled "do not install" (DNI) are not populated by default
+Wire Notes Line
+	6950 6500 6950 6400
+Wire Notes Line
+	6950 6400 11200 6400
 $EndSCHEMATC
