File: mainboard-v05/mainboard.kicad_pcb (KiCad board)
At the start: 4 copper layers, 90.2 x 95.9 mm, 269 parts, among them J1 503182-1852, J10 Conn_01x04, J11 10118194-0001LF, J12 Amphenol_901-144, J13 USB_C_Receptacle_USB2.0, J14 Conn_01x06, J15 Conn_01x02, J16 1985807, J17 1985807, J18 1985807, J2 Conn_01x05, J3 1985807, J4 1985807, J5 Amphenol_901-144, J6 Amphenol_901-144, J7 Amphenol_901-144, J8 Conn_01x09, J9 Conn_01x03, Q1 IRLML2803, Q11 MMDT2907, Q12 BSS138DWQ-7, Q13 BSS138DWQ-7, Q15 MBT2222ADW1T1, Q16 MBT2222ADW1T1, Q17 MMBT2907, Q18 BSS138DWQ-7, Q19 BSS138DWQ-7, Q2 MBT2222ADW1T1, Q20 NDS8434, Q21 NDS8434, Q22 NDS8434, Q3 MBT2222ADW1T1, Q4 IRLML2803, Q5 IRLML2803, Q6 MMBT2222AT, Q7 MBT2222ADW1T1, Q8 MBT2222ADW1T1, SW1 KMR231NG LFS, U1 MAX706RESA, U10 XTB-40, U11 XTB-40, U12 XTB-40, U13 EP2W+, U14 S1216V8, U15 RFM9xBreakout, U16 PE014006, U17 BQ25883RGER, U2 ATSAMD51J19A-AU, U21 TPS7A4501DCQT, U23 RFM98PW, U24 RFM98PW, U3 BMX160, U4 ADM1176-1ARMZ-R7, U5 TPS54226PWPRPWP14_2P31X2P46-L, U6 LTC4121, U7 KF50BD-TR, U8 MR25H40MDF, U9 XTB-40, Y1 32.768kHz

Commit message: tweaking one-shot values for reduced power consumption
Parts:
- R14: value 22.1k -> 22.1K
- R25, R27, R28, R41, R42, R43, R5, R50, R51, R7: value 10k -> 10K
- R29: value 10K -> 73.2K
- R30, R49: value 10K -> 100K
- R32, R33, R6, R60, R92: value 4.7k -> 4.7K
- R39, R40: value 5.1k -> 5.1K
- R47: value 20K -> 200K
Changed lines of the file:
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@@
       (effects (font (size 0.762 0.762) (thickness 0.127)))
     )
-    (fp_text value 4.7k (at 0 1.43 270) (layer F.Fab)
+    (fp_text value 4.7K (at 0 1.43 270) (layer F.Fab)
       (effects (font (size 1 1) (thickness 0.15)))
     )
@@
       (effects (font (size 0.762 0.762) (thickness 0.127)))
     )
-    (fp_text value 4.7k (at 0 1.43) (layer F.Fab)
+    (fp_text value 4.7K (at 0 1.43) (layer F.Fab)
       (effects (font (size 1 1) (thickness 0.15)))
     )
@@
       (effects (font (size 0.762 0.762) (thickness 0.127)) (justify mirror))
     )
-    (fp_text value 10K (at 0 -1.43) (layer B.Fab)
+    (fp_text value 100K (at 0 -1.43) (layer B.Fab)
       (effects (font (size 1 1) (thickness 0.15)) (justify mirror))
     )
@@
       (effects (font (size 0.762 0.762) (thickness 0.127)) (justify mirror))
     )
-    (fp_text value 20K (at 0 -1.43) (layer B.Fab)
+    (fp_text value 200K (at 0 -1.43) (layer B.Fab)
       (effects (font (size 1 1) (thickness 0.15)) (justify mirror))
     )
@@
       (effects (font (size 0.762 0.762) (thickness 0.127)) (justify mirror))
     )
-    (fp_text value 10K (at 0 -1.43) (layer B.Fab)
+    (fp_text value 100K (at 0 -1.43) (layer B.Fab)
       (effects (font (size 1 1) (thickness 0.15)) (justify mirror))
     )
@@
       (effects (font (size 0.762 0.762) (thickness 0.127)) (justify mirror))
     )
-    (fp_text value 10K (at 0 -1.43) (layer B.Fab)
+    (fp_text value 73.2K (at 0 -1.43) (layer B.Fab)
       (effects (font (size 1 1) (thickness 0.15)) (justify mirror))
     )
@@
       (effects (font (size 0.762 0.762) (thickness 0.127)) (justify mirror))
     )
-    (fp_text value 10k (at 0 -1.43) (layer B.Fab)
+    (fp_text value 10K (at 0 -1.43) (layer B.Fab)
       (effects (font (size 1 1) (thickness 0.15)) (justify mirror))
     )
@@
       (effects (font (size 0.762 0.762) (thickness 0.127)) (justify mirror))
     )
-    (fp_text value 10k (at 0 -1.43) (layer B.Fab)
+    (fp_text value 10K (at 0 -1.43) (layer B.Fab)
       (effects (font (size 1 1) (thickness 0.15)) (justify mirror))
     )
@@
       (effects (font (size 0.762 0.762) (thickness 0.127)))
     )
-    (fp_text value 10k (at 0 1.43) (layer F.Fab)
+    (fp_text value 10K (at 0 1.43) (layer F.Fab)
       (effects (font (size 1 1) (thickness 0.15)))
     )
@@
       (effects (font (size 0.762 0.762) (thickness 0.127)))
     )
-    (fp_text value 10k (at 0 1.43) (layer F.Fab)
+    (fp_text value 10K (at 0 1.43) (layer F.Fab)
       (effects (font (size 1 1) (thickness 0.15)))
     )
@@
       (effects (font (size 0.762 0.762) (thickness 0.127)))
     )
-    (fp_text value 10k (at 0 1.43) (layer F.Fab)
+    (fp_text value 10K (at 0 1.43) (layer F.Fab)
       (effects (font (size 1 1) (thickness 0.15)))
     )
@@
       (effects (font (size 0.762 0.762) (thickness 0.127)) (justify mirror))
     )
-    (fp_text value 5.1k (at 0 -1.43 180) (layer B.Fab)
+    (fp_text value 5.1K (at 0 -1.43 180) (layer B.Fab)
       (effects (font (size 1 1) (thickness 0.15)) (justify mirror))
     )
@@
       (effects (font (size 0.762 0.762) (thickness 0.127)) (justify mirror))
     )
-    (fp_text value 5.1k (at 0 -1.43) (layer B.Fab)
+    (fp_text value 5.1K (at 0 -1.43) (layer B.Fab)
       (effects (font (size 1 1) (thickness 0.15)) (justify mirror))
     )
@@
       (effects (font (size 0.762 0.762) (thickness 0.127)))
     )
-    (fp_text value 10k (at 0 1.43) (layer F.Fab)
+    (fp_text value 10K (at 0 1.43) (layer F.Fab)
       (effects (font (size 1 1) (thickness 0.15)))
     )
@@
       (effects (font (size 0.762 0.762) (thickness 0.127)) (justify mirror))
     )
-    (fp_text value 10k (at 0 -1.43 180) (layer B.Fab)
+    (fp_text value 10K (at 0 -1.43 180) (layer B.Fab)
       (effects (font (size 1 1) (thickness 0.15)) (justify mirror))
     )
@@
       (effects (font (size 0.762 0.762) (thickness 0.127)))
     )
-    (fp_text value 10k (at 0 1.43 180) (layer F.Fab)
+    (fp_text value 10K (at 0 1.43 180) (layer F.Fab)
       (effects (font (size 1 1) (thickness 0.15)))
     )
@@
       (effects (font (size 0.762 0.762) (thickness 0.127)))
     )
-    (fp_text value 4.7k (at 0 1.43 270) (layer F.Fab)
+    (fp_text value 4.7K (at 0 1.43 270) (layer F.Fab)
       (effects (font (size 1 1) (thickness 0.15)))
     )
@@
       (effects (font (size 0.762 0.762) (thickness 0.127)))
     )
-    (fp_text value 4.7k (at 0 1.43 90) (layer F.Fab)
+    (fp_text value 4.7K (at 0 1.43 90) (layer F.Fab)
       (effects (font (size 1 1) (thickness 0.15)))
     )
@@
       (effects (font (size 0.762 0.762) (thickness 0.127)))
     )
-    (fp_text value 10k (at 0 1.43 270) (layer F.Fab)
+    (fp_text value 10K (at 0 1.43 270) (layer F.Fab)
       (effects (font (size 1 1) (thickness 0.15)))
     )
@@
       (effects (font (size 0.762 0.762) (thickness 0.127)))
     )
-    (fp_text value 10k (at 0 1.43) (layer F.Fab)
+    (fp_text value 10K (at 0 1.43) (layer F.Fab)
       (effects (font (size 1 1) (thickness 0.15)))
     )
@@
       (effects (font (size 0.635 0.635) (thickness 0.127)))
     )
-    (fp_text value 22.1k (at 0 1.43 90) (layer F.Fab)
+    (fp_text value 22.1K (at 0 1.43 90) (layer F.Fab)
       (effects (font (size 1 1) (thickness 0.15)))
     )
@@
       (effects (font (size 0.635 0.635) (thickness 0.127)))
     )
-    (fp_text value 4.7k (at 0 1.43 270) (layer F.Fab)
+    (fp_text value 4.7K (at 0 1.43 270) (layer F.Fab)
       (effects (font (size 1 1) (thickness 0.15)))
     )
